File: Hardware/InkTime.sch (EAGLE design)
At the start: 105 parts, among them IC1 BQ25180YBGR_BQ25180YBGRBBQ, IC2 DRV2605YZFR, IC3 BMA421, IC9 RT6160AWSC, J1 503480-2400, J2 TC2030-IDC, J4 KH-TYPE-C-16P, Q1 ESP32_C6_LIBRARY_4_ESP32_WROV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, Q3 SI1308EDL-T1-GE3, U3 MAX17048G+T10, X1 32MHz, X2 32.768kHz

Commit message: Fixed minor schematic and board issues
Parts:
- Q1: value ESP32_C6_LIBRARY_4_ESP32_WROVER_SPARKFUN-DISCRETESEMI_MOSFET_PCH -> DMG2305UX-7
- renumbered U$1 to U1
